File: kicad/gpsdo.sch (KiCad schematic (older format))
At the start: 1 part

Commit message: add skeleton kicad project
Parts:
- added J?: RJ45_Abracon_ARJP11A-MASA-B-A-EMU2, Connector_RJ:RJ45_Abracon_ARJP11A-MA_Horizontal, symbol Connector:RJ45_Abracon_ARJP11A-MASA-B-A-EMU2
- added U1: 549CAAC000111BBG, Oscillator:Oscillator_SMD_SI570_SI571_Standard, symbol Oscillator:Si570
- added U2: MAX-8Q, RF_GPS:ublox_MAX, symbol RF_GPS:MAX-8Q
- added U3: Si7051-A20, Package_DFN_QFN:DFN-6-1EP_3x3mm_P1mm_EP1.65x2.55mm, symbol Sensor_Temperature:Si7051-A20
Connections:
- net labels added: GND
- wire segments 0 -> 3
Changed lines of the file:
@@
 U 1 1 60FAE182
 P 8350 5150
-F 0 "U?" H 8350 2461 50  0000 C CNN
-F 1 "PIC32MX795F512L-80x-PF" H 8350 2370 50  0000 C CNN
+F 0 "U?" H 7750 2600 50  0000 C CNN
+F 1 "PIC32MX795F512L-80x-PF" H 9100 2600 50  0000 C CNN
 F 2 "Package_QFP:TQFP-100_14x14mm_P0.5mm" H 8350 2150 50  0001 C CNN
 F 3 "http://ww1.microchip.com/downloads/en/DeviceDoc/60001156J.pdf" H 8350 2150 50  0001 C CNN
@@
 	1    0    0    -1
 $EndComp
+$Comp
+L Oscillator:Si570 U1
+U 1 1 60FCFECF
+P 4050 4950
+F 0 "U1" H 3700 5350 50  0000 C CNN
+F 1 "549CAAC000111BBG" H 4500 4550 50  0000 C CNN
+F 2 "Oscillator:Oscillator_SMD_SI570_SI571_Standard" H 4050 4650 50  0001 C CNN
+F 3 "http://www.silabs.com/Support%20Documents/TechnicalDocs/si570.pdf" H 3650 5650 50  0001 C CNN
+	1    4050 4950
+	1    0    0    -1
+$EndComp
+$Comp
+L RF_GPS:MAX-8Q U2
+U 1 1 60FD23E0
+P 4050 3000
+F 0 "U2" H 4250 2350 50  0000 C CNN
+F 1 "MAX-8Q" H 4350 2250 50  0000 C CNN
+F 2 "RF_GPS:ublox_MAX" H 4450 2350 50  0001 C CNN
+F 3 "https://www.u-blox.com/sites/default/files/MAX-8_DataSheet_%28UBX-16000093%29.pdf" H 4050 3000 50  0001 C CNN
+	1    4050 3000
+	1    0    0    -1
+$EndComp
+$Comp
+L Sensor_Temperature:Si7051-A20 U3
+U 1 1 60FD391B
+P 4050 6050
+F 0 "U3" H 4394 6096 50  0000 L CNN
+F 1 "Si7051-A20" H 4394 6005 50  0000 L CNN
+F 2 "Package_DFN_QFN:DFN-6-1EP_3x3mm_P1mm_EP1.65x2.55mm" H 4050 5650 50  0001 C CNN
+F 3 "https://www.silabs.com/documents/public/data-sheets/Si7050-1-3-4-5-A20.pdf" H 3850 6350 50  0001 C CNN
+	1    4050 6050
+	1    0    0    -1
+$EndComp
+$Comp
+L Connector:RJ45_Abracon_ARJP11A-MASA-B-A-EMU2 J?
+U 1 1 60FD505B
+P 15250 2450
+F 0 "J?" H 15250 3967 50  0000 C CNN
+F 1 "RJ45_Abracon_ARJP11A-MASA-B-A-EMU2" H 15250 3876 50  0000 C CNN
+F 2 "Connector_RJ:RJ45_Abracon_ARJP11A-MA_Horizontal" H 15250 3850 50  0001 C CNN
+F 3 "https://abracon.com/Magnetics/lan/ARJP11A.PDF" H 15100 1600 50  0001 C CNN
+	1    15250 2450
+	1    0    0    -1
+$EndComp
+$Comp
+L power:GND #PWR?
+U 1 1 60FDC4EE
+P 14550 2150
+F 0 "#PWR?" H 14550 1900 50  0001 C CNN
+F 1 "GND" V 14555 2022 50  0000 R CNN
+F 2 "" H 14550 2150 50  0001 C CNN
+F 3 "" H 14550 2150 50  0001 C CNN
+	1    14550 2150
+	0    1    1    0
+$EndComp
+$Comp
+L power:GND #PWR?
+U 1 1 60FDFB2F
+P 4050 6350
+F 0 "#PWR?" H 4050 6100 50  0001 C CNN
+F 1 "GND" H 4055 6177 50  0000 C CNN
+F 2 "" H 4050 6350 50  0001 C CNN
+F 3 "" H 4050 6350 50  0001 C CNN
+	1    4050 6350
+	1    0    0    -1
+$EndComp
+$Comp
+L power:GND #PWR?
+U 1 1 60FDFF77
+P 4050 5350
+F 0 "#PWR?" H 4050 5100 50  0001 C CNN
+F 1 "GND" H 4055 5177 50  0000 C CNN
+F 2 "" H 4050 5350 50  0001 C CNN
+F 3 "" H 4050 5350 50  0001 C CNN
+	1    4050 5350
+	1    0    0    -1
+$EndComp
+$Comp
+L power:GND #PWR?
+U 1 1 60FE03FF
+P 4050 3700
+F 0 "#PWR?" H 4050 3450 50  0001 C CNN
+F 1 "GND" H 4055 3527 50  0000 C CNN
+F 2 "" H 4050 3700 50  0001 C CNN
+F 3 "" H 4050 3700 50  0001 C CNN
+	1    4050 3700
+	1    0    0    -1
+$EndComp
+Wire Wire Line
+	4550 4850 5600 4850
+Wire Wire Line
+	5600 4850 5600 4550
+Wire Wire Line
+	5600 4550 7150 4550
+$Comp
+L power:GND #PWR?
+U 1 1 60FE526E
+P 8250 7750
+F 0 "#PWR?" H 8250 7500 50  0001 C CNN
+F 1 "GND" H 8255 7577 50  0000 C CNN
+F 2 "" H 8250 7750 50  0001 C CNN
+F 3 "" H 8250 7750 50  0001 C CNN
+	1    8250 7750
+	1    0    0    -1
+$EndComp
+$Comp
+L power:GND #PWR?
+U 1 1 60FE55A2
+P 8450 7750
+F 0 "#PWR?" H 8450 7500 50  0001 C CNN
+F 1 "GND" H 8455 7577 50  0000 C CNN
+F 2 "" H 8450 7750 50  0001 C CNN
+F 3 "" H 8450 7750 50  0001 C CNN
+	1    8450 7750
+	1    0    0    -1
+$EndComp

Commit message: add skeleton kicad project
Parts:
- added C2: 10n, Capacitor_SMD:C_0805_2012Metric, symbol Device:C_Small
- added J2: Conn_Coaxial, Connector_Coaxial:SMA_Molex_73251-1153_EdgeMount_Horizontal, symbol Connector:Conn_Coaxial
- added L1: 27n, Inductor_SMD:L_0805_2012Metric, symbol Device:L_Small
- added R1: 10, Resistor_SMD:R_0805_2012Metric, symbol Device:R_Small_US
- U3: footprint Package_DFN_QFN:DFN-6-1EP_3x3mm_P1mm_EP1.65x2.55mm -> Package_DFN_QFN:DFN-6-1EP_3x3mm_P1mm_EP1.5x2.4mm
- gave numbers to parts that had none: 2
Connections:
- net labels added: +3.3V
- wire segments 3 -> 24
Other:
- moved on the sheet: U3
Changed lines of the file:
@@
 $EndDescr
 $Comp
-L MCU_Microchip_PIC32:PIC32MX795F512L-80x-PF U?
+L MCU_Microchip_PIC32:PIC32MX795F512L-80x-PF U4
 U 1 1 60FAE182
 P 8350 5150
-F 0 "U?" H 7750 2600 50  0000 C CNN
+F 0 "U4" H 7750 2600 50  0000 C CNN
 F 1 "PIC32MX795F512L-80x-PF" H 9100 2600 50  0000 C CNN
 F 2 "Package_QFP:TQFP-100_14x14mm_P0.5mm" H 8350 2150 50  0001 C CNN
@@
 L Sensor_Temperature:Si7051-A20 U3
 U 1 1 60FD391B
-P 4050 6050
-F 0 "U3" H 4394 6096 50  0000 L CNN
-F 1 "Si7051-A20" H 4394 6005 50  0000 L CNN
-F 2 "Package_DFN_QFN:DFN-6-1EP_3x3mm_P1mm_EP1.65x2.55mm" H 4050 5650 50  0001 C CNN
-F 3 "https://www.silabs.com/documents/public/data-sheets/Si7050-1-3-4-5-A20.pdf" H 3850 6350 50  0001 C CNN
-	1    4050 6050
-	1    0    0    -1
-$EndComp
-$Comp
-L Connector:RJ45_Abracon_ARJP11A-MASA-B-A-EMU2 J?
+P 4050 6150
+F 0 "U3" H 4394 6196 50  0000 L CNN
+F 1 "Si7051-A20" H 4394 6105 50  0000 L CNN
+F 2 "Package_DFN_QFN:DFN-6-1EP_3x3mm_P1mm_EP1.5x2.4mm" H 4050 5750 50  0001 C CNN
+F 3 "https://www.silabs.com/documents/public/data-sheets/Si7050-1-3-4-5-A20.pdf" H 3850 6450 50  0001 C CNN
+	1    4050 6150
+	1    0    0    -1
+$EndComp
+$Comp
+L Connector:RJ45_Abracon_ARJP11A-MASA-B-A-EMU2 J1
 U 1 1 60FD505B
 P 15250 2450
-F 0 "J?" H 15250 3967 50  0000 C CNN
+F 0 "J1" H 15250 3967 50  0000 C CNN
 F 1 "RJ45_Abracon_ARJP11A-MASA-B-A-EMU2" H 15250 3876 50  0000 C CNN
 F 2 "Connector_RJ:RJ45_Abracon_ARJP11A-MA_Horizontal" H 15250 3850 50  0001 C CNN
@@
 $EndComp
 $Comp
-L power:GND #PWR?
+L power:GND #PWR0101
 U 1 1 60FDC4EE
 P 14550 2150
-F 0 "#PWR?" H 14550 1900 50  0001 C CNN
+F 0 "#PWR0101" H 14550 1900 50  0001 C CNN
 F 1 "GND" V 14555 2022 50  0000 R CNN
 F 2 "" H 14550 2150 50  0001 C CNN
@@
 $EndComp
 $Comp
-L power:GND #PWR?
+L power:GND #PWR0102
 U 1 1 60FDFB2F
-P 4050 6350
-F 0 "#PWR?" H 4050 6100 50  0001 C CNN
-F 1 "GND" H 4055 6177 50  0000 C CNN
-F 2 "" H 4050 6350 50  0001 C CNN
-F 3 "" H 4050 6350 50  0001 C CNN
-	1    4050 6350
-	1    0    0    -1
-$EndComp
-$Comp
-L power:GND #PWR?
+P 4050 6450
+F 0 "#PWR0102" H 4050 6200 50  0001 C CNN
+F 1 "GND" H 4055 6277 50  0000 C CNN
+F 2 "" H 4050 6450 50  0001 C CNN
+F 3 "" H 4050 6450 50  0001 C CNN
+	1    4050 6450
+	1    0    0    -1
+$EndComp
+$Comp
+L power:GND #PWR0103
 U 1 1 60FDFF77
 P 4050 5350
-F 0 "#PWR?" H 4050 5100 50  0001 C CNN
+F 0 "#PWR0103" H 4050 5100 50  0001 C CNN
 F 1 "GND" H 4055 5177 50  0000 C CNN
 F 2 "" H 4050 5350 50  0001 C CNN
@@
 $EndComp
 $Comp
-L power:GND #PWR?
+L power:GND #PWR0104
 U 1 1 60FE03FF
 P 4050 3700
-F 0 "#PWR?" H 4050 3450 50  0001 C CNN
+F 0 "#PWR0104" H 4050 3450 50  0001 C CNN
 F 1 "GND" H 4055 3527 50  0000 C CNN
 F 2 "" H 4050 3700 50  0001 C CNN
@@
 	5600 4550 7150 4550
 $Comp
-L power:GND #PWR?
+L power:GND #PWR0105
 U 1 1 60FE526E
 P 8250 7750
-F 0 "#PWR?" H 8250 7500 50  0001 C CNN
+F 0 "#PWR0105" H 8250 7500 50  0001 C CNN
 F 1 "GND" H 8255 7577 50  0000 C CNN
 F 2 "" H 8250 7750 50  0001 C CNN
@@
 $EndComp
 $Comp
-L power:GND #PWR?
+L power:GND #PWR0106
 U 1 1 60FE55A2
 P 8450 7750
-F 0 "#PWR?" H 8450 7500 50  0001 C CNN
+F 0 "#PWR0106" H 8450 7500 50  0001 C CNN
 F 1 "GND" H 8455 7577 50  0000 C CNN
 F 2 "" H 8450 7750 50  0001 C CNN
@@
 	1    0    0    -1
 $EndComp
+Wire Wire Line
+	3550 5050 3300 5050
+Wire Wire Line
+	3300 6150 3650 6150
+Wire Wire Line
+	3650 6050 3400 6050
+Wire Wire Line
+	3400 5150 3550 5150
+$Comp
+L power:+3.3V #PWR0107
+U 1 1 60FB36E1
+P 4050 5850
+F 0 "#PWR0107" H 4050 5700 50  0001 C CNN
+F 1 "+3.3V" H 4065 6023 50  0000 C CNN
+F 2 "" H 4050 5850 50  0001 C CNN
+F 3 "" H 4050 5850 50  0001 C CNN
+	1    4050 5850
+	1    0    0    -1
+$EndComp
+$Comp
+L power:+3.3V #PWR0108
+U 1 1 60FB3C13
+P 4050 4550
+F 0 "#PWR0108" H 4050 4400 50  0001 C CNN
+F 1 "+3.3V" H 4065 4723 50  0000 C CNN
+F 2 "" H 4050 4550 50  0001 C CNN
+F 3 "" H 4050 4550 50  0001 C CNN
+	1    4050 4550
+	1    0    0    -1
+$EndComp
+Wire Wire Line
+	3300 5050 3300 6150
+Wire Wire Line
+	3400 5150 3400 6050
+Wire Notes Line
+	2850 4200 5250 4200
+Wire Notes Line
+	5250 4200 5250 6850
+Wire Notes Line
+	5250 6850 2850 6850
+Wire Notes Line
+	2850 6850 2850 4200
+$Comp
+L Connector:Conn_Coaxial J2
+U 1 1 60FBD0FE
+P 5150 3000
+F 0 "J2" H 5250 2975 50  0000 L CNN
+F 1 "Conn_Coaxial" H 5250 2884 50  0000 L CNN
+F 2 "Connector_Coaxial:SMA_Molex_73251-1153_EdgeMount_Horizontal" H 5150 3000 50  0001 C CNN
+F 3 " ~" H 5150 3000 50  0001 C CNN
+	1    5150 3000
+	1    0    0    -1
+$EndComp
+$Comp
+L power:GND #PWR0109
+U 1 1 60FBDB7E
+P 5150 3200
+F 0 "#PWR0109" H 5150 2950 50  0001 C CNN
+F 1 "GND" H 5155 3027 50  0000 C CNN
+F 2 "" H 5150 3200 50  0001 C CNN
+F 3 "" H 5150 3200 50  0001 C CNN
+	1    5150 3200
+	1    0    0    -1
+$EndComp
+$Comp
+L Device:L_Small L1
+U 1 1 60FBF33B
+P 4850 2750
+F 0 "L1" H 4898 2796 50  0000 L CNN
+F 1 "27n" H 4898 2705 50  0000 L CNN
+F 2 "Inductor_SMD:L_0805_2012Metric" H 4850 2750 50  0001 C CNN
+F 3 "~" H 4850 2750 50  0001 C CNN
+	1    4850 2750
+	1    0    0    -1
+$EndComp
+Wire Wire Line
+	4850 2850 4850 3000
+Connection ~ 4850 3000
+Wire Wire Line
+	4850 3000 4950 3000
+$Comp
+L Device:C_Small C2
+U 1 1 60FC1266
+P 5000 2550
+F 0 "C2" V 4771 2550 50  0000 C CNN
+F 1 "10n" V 4862 2550 50  0000 C CNN
+F 2 "Capacitor_SMD:C_0805_2012Metric" H 5000 2550 50  0001 C CNN
+F 3 "~" H 5000 2550 50  0001 C CNN
+	1    5000 2550
+	0    1    1    0
+$EndComp
+Connection ~ 4850 2550
+Wire Wire Line
+	4850 2550 4850 2650
+Wire Wire Line
+	4900 2550 4850 2550
+$Comp
+L power:GND #PWR0112
+U 1 1 60FC3F9C
+P 5100 2550
+F 0 "#PWR0112" H 5100 2300 50  0001 C CNN
+F 1 "GND" V 5105 2422 50  0000 R CNN
+F 2 "" H 5100 2550 50  0001 C CNN
+F 3 "" H 5100 2550 50  0001 C CNN
+	1    5100 2550
+	0    -1   -1   0
+$EndComp
+$Comp
+L power:+3.3V #PWR0110
+U 1 1 60FD182D
+P 3950 2200
+F 0 "#PWR0110" H 3950 2050 50  0001 C CNN
+F 1 "+3.3V" H 3965 2373 50  0000 C CNN
+F 2 "" H 3950 2200 50  0001 C CNN
+F 3 "" H 3950 2200 50  0001 C CNN
+	1    3950 2200
+	1    0    0    -1
+$EndComp
+Wire Wire Line
+	3950 2200 3950 2250
+Wire Wire Line
+	4050 2300 4050 2250
+Wire Wire Line
+	4050 2250 3950 2250
+Connection ~ 3950 2250
+Wire Wire Line
+	3950 2250 3950 2300
+Wire Wire Line
+	3850 2300 3850 2250
+Wire Wire Line
+	3850 2250 3950 2250
+Wire Wire Line
+	4250 2300 4250 2250
+Wire Wire Line
+	4850 2250 4850 2550
+Wire Wire Line
+	4650 3000 4850 3000
+$Comp
+L Device:R_Small_US R1
+U 1 1 60FDF5E7
+P 4650 2250
+F 0 "R1" V 4445 2250 50  0000 C CNN
+F 1 "10" V 4536 2250 50  0000 C CNN
+F 2 "Resistor_SMD:R_0805_2012Metric" H 4650 2250 50  0001 C CNN
+F 3 "~" H 4650 2250 50  0001 C CNN
+	1    4650 2250
+	0    1    1    0
+$EndComp
+Wire Wire Line
+	4750 2250 4850 2250
+Wire Wire Line
+	4550 2250 4250 2250
 $EndSCHEMATC

Commit message: add ethernet phy
Parts:
- added C2, C3, C4, C5: 100n, Capacitor_SMD:C_0805_2012Metric, symbol Device:C_Small
- added R2, R3: 100, Resistor_SMD:R_0805_2012Metric, symbol Device:R_Small_US
- added U5: DP83640TVV_NOPB, Package_QFP:LQFP-48_7x7mm_P0.5mm, symbol DP83640TVV_NOPB:DP83640TVV_NOPB
- renumbered C2 to C1
Connections:
- net labels added: RD+, RD-, TD+, TD-
- wire segments 24 -> 48
Other:
- moved on the sheet: C1, J1, J2, L1, R1, U1, U2, U3

Commit message: board progress
Parts:
- removed U4: PIC32MX795F512L-80x-PF, Package_QFP:TQFP-100_14x14mm_P0.5mm, symbol MCU_Microchip_PIC32:PIC32MX795F512L-80x-PF
- added R10, R11, R12, R13, R14, R15, R16, R17, R18, R19, R4, R5, R6, R7, R8, R9: 10k, Resistor_SMD:R_0603_1608Metric, symbol Device:R_Small_US
- added U5: AM3352BZCE60, kicad:BGA298C65P19X19_1300X1300X130, symbol AM3352BZCE60:AM3352BZCE60
- renumbered C4 to C2, C5 to C3, C2 to C4, C3 to C5, J2 to J1, J1 to J2, U3 to U2, U2 to U3, U5 to U4
Connections:
- net labels added: CLK_25M
- wire segments 48 -> 75
Other:
- note added: "SYSBOOT = 0100 0000 0001 0111 b"

Commit message: update layout
Parts:
- removed C3: 100n, Capacitor_SMD:C_0805_2012Metric, symbol Device:C_Small
- removed J2: RJ45_Abracon_ARJP11A-MASA-B-A-EMU2, Connector_RJ:RJ45_Abracon_ARJP11A-MA_Horizontal, symbol Connector:RJ45_Abracon_ARJP11A-MASA-B-A-EMU2
- removed R10, R11, R12, R13, R14, R15, R16, R17, R18, R19, R4, R5, R6, R7, R8, R9: 10k, Resistor_SMD:R_0603_1608Metric, symbol Device:R_Small_US
- removed R2, R3: 100, Resistor_SMD:R_0805_2012Metric, symbol Device:R_Small_US
- removed U4: DP83640TVV_NOPB, Package_QFP:LQFP-48_7x7mm_P0.5mm, symbol DP83640TVV_NOPB:DP83640TVV_NOPB
- removed U5: AM3352BZCE60, kicad:BGA298C65P19X19_1300X1300X130, symbol AM3352BZCE60:AM3352BZCE60
- added C5, C6: 100n, Capacitor_SMD:C_0805_2012Metric, symbol Device:C_Small
- added C7: 470n, Capacitor_SMD:C_0805_2012Metric, symbol Device:C_Small
- added U1: MSP430F5171IDA, Package_SO:TSSOP-38_4.4x9.7mm_P0.5mm, symbol 2021-07-26_01-49-48:MSP430F5171IDA
- renumbered C4 to C3, C5 to C4, U3 to U2, U1 to U3, U2 to U4
Connections:
- net labels removed: RD+, RD-, TD+, TD-
- wire segments 75 -> 27
Other:
- note removed: "SYSBOOT = 0100 0000 0001 0111 b"
- moved on the sheet: C1, C3, C4, J1, L1, R1, U2, U3, U4

Commit message: update layout
Parts:
- added J2, J3, J4, J5: Conn_01x04_Male, Connector_PinHeader_2.54mm:PinHeader_1x04_P2.54mm_Vertical, symbol Connector:Conn_01x04_Male
Connections:
- net GND: now also J2.1 (Pin_1), J2.2 (Pin_2), J2.3 (Pin_3), J2.4 (Pin_4), J3.1 (Pin_1), J3.2 (Pin_2), J3.3 (Pin_3), J3.4 (Pin_4), J4.1 (Pin_1), J4.2 (Pin_2), J4.3 (Pin_3), J4.4 (Pin_4), J5.1 (Pin_1), J5.2 (Pin_2), J5.3 (Pin_3), J5.4 (Pin_4)
- net gPPS: now reaches U2.4 (TIMEPULSE)
- net gPPS: now also U1.15 (P1-6/PM_TD0-0)
- net oPPS: now reaches U1.16 (P1-7/PM_TD0-1)
- net ePPS: now reaches U1.17 (P2-0/PM_TD0-2)
Changed lines of the file:
@@
 Text GLabel 1600 1300 0    50   Input ~ 0
 CLK_25M
+Text GLabel 1700 7250 0    50   Input ~ 0
+gPPS
+Text GLabel 1600 2600 0    50   Input ~ 0
+gPPS
+$Comp
+L Connector:Conn_01x04_Male J2
+U 1 1 61001312
+P 9650 4550
+F 0 "J2" H 9758 4831 50  0000 C CNN
+F 1 "Conn_01x04_Male" H 9758 4740 50  0000 C CNN
+F 2 "Connector_PinHeader_2.54mm:PinHeader_1x04_P2.54mm_Vertical" H 9650 4550 50  0001 C CNN
+F 3 "~" H 9650 4550 50  0001 C CNN
+	1    9650 4550
+	1    0    0    -1
+$EndComp
+$Comp
+L power:GND #PWR0101
+U 1 1 61004A66
+P 9850 4450
+F 0 "#PWR0101" H 9850 4200 50  0001 C CNN
+F 1 "GND" V 9850 4250 50  0000 C CNN
+F 2 "" H 9850 4450 50  0001 C CNN
+F 3 "" H 9850 4450 50  0001 C CNN
+	1    9850 4450
+	0    -1   -1   0
+$EndComp
+$Comp
+L power:GND #PWR0102
+U 1 1 61004F29
+P 9850 4550
+F 0 "#PWR0102" H 9850 4300 50  0001 C CNN
+F 1 "GND" V 9850 4350 50  0000 C CNN
+F 2 "" H 9850 4550 50  0001 C CNN
+F 3 "" H 9850 4550 50  0001 C CNN
+	1    9850 4550
+	0    -1   -1   0
+$EndComp
+$Comp
+L power:GND #PWR0103
+U 1 1 6100517B
+P 9850 4650
+F 0 "#PWR0103" H 9850 4400 50  0001 C CNN
+F 1 "GND" V 9850 4450 50  0000 C CNN
+F 2 "" H 9850 4650 50  0001 C CNN
+F 3 "" H 9850 4650 50  0001 C CNN
+	1    9850 4650
+	0    -1   -1   0
+$EndComp
+$Comp
+L power:GND #PWR0104
+U 1 1 61005419
+P 9850 4750
+F 0 "#PWR0104" H 9850 4500 50  0001 C CNN
+F 1 "GND" V 9850 4550 50  0000 C CNN
+F 2 "" H 9850 4750 50  0001 C CNN
+F 3 "" H 9850 4750 50  0001 C CNN
+	1    9850 4750
+	0    -1   -1   0
+$EndComp
+$Comp
+L Connector:Conn_01x04_Male J3
+U 1 1 61012471
+P 9650 5150
+F 0 "J3" H 9758 5431 50  0000 C CNN
+F 1 "Conn_01x04_Male" H 9758 5340 50  0000 C CNN
+F 2 "Connector_PinHeader_2.54mm:PinHeader_1x04_P2.54mm_Vertical" H 9650 5150 50  0001 C CNN
+F 3 "~" H 9650 5150 50  0001 C CNN
+	1    9650 5150
+	1    0    0    -1
+$EndComp
+$Comp
+L power:GND #PWR0105
+U 1 1 61012477
+P 9850 5050
+F 0 "#PWR0105" H 9850 4800 50  0001 C CNN
+F 1 "GND" V 9850 4850 50  0000 C CNN
+F 2 "" H 9850 5050 50  0001 C CNN
+F 3 "" H 9850 5050 50  0001 C CNN
+	1    9850 5050
+	0    -1   -1   0
+$EndComp
+$Comp
+L power:GND #PWR0106
+U 1 1 6101247D
+P 9850 5150
+F 0 "#PWR0106" H 9850 4900 50  0001 C CNN
+F 1 "GND" V 9850 4950 50  0000 C CNN
+F 2 "" H 9850 5150 50  0001 C CNN
+F 3 "" H 9850 5150 50  0001 C CNN
+	1    9850 5150
+	0    -1   -1   0
+$EndComp
+$Comp
+L power:GND #PWR0107
+U 1 1 61012483
+P 9850 5250
+F 0 "#PWR0107" H 9850 5000 50  0001 C CNN
+F 1 "GND" V 9850 5050 50  0000 C CNN
+F 2 "" H 9850 5250 50  0001 C CNN
+F 3 "" H 9850 5250 50  0001 C CNN
+	1    9850 5250
+	0    -1   -1   0
+$EndComp
+$Comp
+L power:GND #PWR0108
+U 1 1 61012489
+P 9850 5350
+F 0 "#PWR0108" H 9850 5100 50  0001 C CNN
+F 1 "GND" V 9850 5150 50  0000 C CNN
+F 2 "" H 9850 5350 50  0001 C CNN
+F 3 "" H 9850 5350 50  0001 C CNN
+	1    9850 5350
+	0    -1   -1   0
+$EndComp
+$Comp
+L Connector:Conn_01x04_Male J4
+U 1 1 61013E1B
+P 9650 5750
+F 0 "J4" H 9758 6031 50  0000 C CNN
+F 1 "Conn_01x04_Male" H 9758 5940 50  0000 C CNN
+F 2 "Connector_PinHeader_2.54mm:PinHeader_1x04_P2.54mm_Vertical" H 9650 5750 50  0001 C CNN
+F 3 "~" H 9650 5750 50  0001 C CNN
+	1    9650 5750
+	1    0    0    -1
+$EndComp
+$Comp
+L power:GND #PWR0109
+U 1 1 61013E21
+P 9850 5650
+F 0 "#PWR0109" H 9850 5400 50  0001 C CNN
+F 1 "GND" V 9850 5450 50  0000 C CNN
+F 2 "" H 9850 5650 50  0001 C CNN
+F 3 "" H 9850 5650 50  0001 C CNN
+	1    9850 5650
+	0    -1   -1   0
+$EndComp
+$Comp
+L power:GND #PWR0110
+U 1 1 61013E27
+P 9850 5750
+F 0 "#PWR0110" H 9850 5500 50  0001 C CNN
+F 1 "GND" V 9850 5550 50  0000 C CNN
+F 2 "" H 9850 5750 50  0001 C CNN
+F 3 "" H 9850 5750 50  0001 C CNN
+	1    9850 5750
+	0    -1   -1   0
+$EndComp
+$Comp
+L power:GND #PWR0111
+U 1 1 61013E2D
+P 9850 5850
+F 0 "#PWR0111" H 9850 5600 50  0001 C CNN
+F 1 "GND" V 9850 5650 50  0000 C CNN
+F 2 "" H 9850 5850 50  0001 C CNN
+F 3 "" H 9850 5850 50  0001 C CNN
+	1    9850 5850
+	0    -1   -1   0
+$EndComp
+$Comp
+L power:GND #PWR0112
+U 1 1 61013E33
+P 9850 5950
+F 0 "#PWR0112" H 9850 5700 50  0001 C CNN
+F 1 "GND" V 9850 5750 50  0000 C CNN
+F 2 "" H 9850 5950 50  0001 C CNN
+F 3 "" H 9850 5950 50  0001 C CNN
+	1    9850 5950
+	0    -1   -1   0
+$EndComp
+$Comp
+L Connector:Conn_01x04_Male J5
+U 1 1 61014761
+P 9650 6350
+F 0 "J5" H 9758 6631 50  0000 C CNN
+F 1 "Conn_01x04_Male" H 9758 6540 50  0000 C CNN
+F 2 "Connector_PinHeader_2.54mm:PinHeader_1x04_P2.54mm_Vertical" H 9650 6350 50  0001 C CNN
+F 3 "~" H 9650 6350 50  0001 C CNN
+	1    9650 6350
+	1    0    0    -1
+$EndComp
+$Comp
+L power:GND #PWR0113
+U 1 1 61014767
+P 9850 6250
+F 0 "#PWR0113" H 9850 6000 50  0001 C CNN
+F 1 "GND" V 9850 6050 50  0000 C CNN
+F 2 "" H 9850 6250 50  0001 C CNN
+F 3 "" H 9850 6250 50  0001 C CNN
+	1    9850 6250
+	0    -1   -1   0
+$EndComp
+$Comp
+L power:GND #PWR0114
+U 1 1 6101476D
+P 9850 6350
+F 0 "#PWR0114" H 9850 6100 50  0001 C CNN
+F 1 "GND" V 9850 6150 50  0000 C CNN
+F 2 "" H 9850 6350 50  0001 C CNN
+F 3 "" H 9850 6350 50  0001 C CNN
+	1    9850 6350
+	0    -1   -1   0
+$EndComp
+$Comp
+L power:GND #PWR0115
+U 1 1 61014773
+P 9850 6450
+F 0 "#PWR0115" H 9850 6200 50  0001 C CNN
+F 1 "GND" V 9850 6250 50  0000 C CNN
+F 2 "" H 9850 6450 50  0001 C CNN
+F 3 "" H 9850 6450 50  0001 C CNN
+	1    9850 6450
+	0    -1   -1   0
+$EndComp
+$Comp
+L power:GND #PWR0116
+U 1 1 61014779
+P 9850 6550
+F 0 "#PWR0116" H 9850 6300 50  0001 C CNN
+F 1 "GND" V 9850 6350 50  0000 C CNN
+F 2 "" H 9850 6550 50  0001 C CNN
+F 3 "" H 9850 6550 50  0001 C CNN
+	1    9850 6550
+	0    -1   -1   0
+$EndComp
+Text GLabel 1600 2700 0    50   Input ~ 0
+oPPS
+Text GLabel 1600 2800 0    50   Input ~ 0
+ePPS
 $EndSCHEMATC

Commit message: update board layout
Parts:
- added C10: 10u, Capacitor_SMD:C_0805_2012Metric, symbol Device:C_Small
- added C11, C8, C9: 100n, Resistor_SMD:R_0603_1608Metric, symbol Device:C_Small
- added R2, R3, R4, R5, R6, R7: 1.5k, Resistor_SMD:R_0603_1608Metric, symbol Device:R_Small_US
- added U5: LTC4317, Package_DFN_QFN:DFN-16-1EP_3x5mm_P0.5mm_EP1.66x4.4mm, symbol Interface:LTC4317
- C1, C2, C3, C4, C5, C6: footprint Capacitor_SMD:C_0805_2012Metric -> Resistor_SMD:R_0603_1608Metric
- L1: footprint Inductor_SMD:L_0805_2012Metric -> Resistor_SMD:R_0603_1608Metric
- R1: footprint Resistor_SMD:R_0805_2012Metric -> Resistor_SMD:R_0603_1608Metric
Connections:
- net +3V3: now also J2.3 (Pin_3), U3.1 (NC), U4.4 (NC), C10.1, C11.1, C8.1, C9.1, R2.1, R3.2, R4.1, R5.2, R6.1, R7.2, U5.3 (XORH2), U5.4 (XORL2), U5.5 (XORH1), U5.6 (XORL1), U5.7 (VCC)
- net GND: now also C10.2, C11.2, C8.2, C9.2, U5.1 (GND), U5.17 (EP); no longer J2.3 (Pin_3), J2.4 (Pin_4), J4.1 (Pin_1), J4.2 (Pin_2), J5.1 (Pin_1), J5.2 (Pin_2)
- net ePPS: now also J2.4 (Pin_4)
- net at U3.7 (SDA), U4.1 (SDA): now also R7.1, U5.13 (SDAOUT1); no longer U2.16 (SDA)
- net at U3.8 (SCL), U4.6 (SCL): now also R6.2, U5.14 (SCLOUT1); no longer U2.17 (SCL)
- net at U2.2 (TXD): now also J5.1 (Pin_1)
- net at U2.3 (RXD): now also J5.2 (Pin_2)
- net at U2.9 (~RESET): now also U1.19 (P2-2/PM_TD1-1)
- net at U1.10 (P1-5/PM_UCB0SOMI/PM_UCB0SCL/A5*/CB5): now also R2.2, U5.15 (SCLIN)
- net at U1.23 (P2-4/PM_TEC0CLR/PM_TEC0FLT2_/PM_TD0-0): now also U5.2 (ENABLE2)
- net at U1.24 (P2-5/PM_TEC0FLT0/PM_TD0-1): now also U5.8 (ENABLE1)
- net at U1.6 (P1-1/PM_UCA0TXD/PM_UCA0SIMO/A1*/CB1): now also J4.1 (Pin_1)
- net at U1.7 (P1-2/PM_UCA0RXD/PM_UCA0SOMI/A2*/CB2): now also J4.2 (Pin_2)
- net at U1.9 (P1-4/PM_UCB0SIMO/PM_UCB0SDA/A4*/CB4): now also R3.1, U5.12 (SDAIN)
- new net: R5.1, U2.16 (SDA), U5.11 (SDAOUT2)
- new net: R4.2, U2.17 (SCL), U5.16 (SCLOUT2)
Other:
- moved on the sheet: C2, C5, C6, J4, J5
