File: kicad/gpsdo.sch (KiCad schematic (older format))
At the start: 29 parts, among them J1 Conn_Coaxial, J2 Conn_01x04_Male, J3 Conn_01x04_Male, J4 Conn_01x04_Male, J5 Conn_01x04_Male, U1 MSP430F5171IDA, U2 MAX-8Q, U3 549CAAC000111BBG, U4 Si7051-A20, U5 LTC4317

Commit message: update pcb layout
Parts:
- added C12, C13, C14, C15: 100n, Resistor_SMD:R_0603_1608Metric, symbol Device:C_Small
- added J6: Conn_01x04_Male, Connector_PinHeader_2.54mm:PinHeader_1x04_P2.54mm_Vertical, symbol Connector:Conn_01x04_Male
- added R8, R9: 15k, Resistor_SMD:R_0603_1608Metric, symbol Device:R_Small_US
- added U10, U8: 74AUC1G79, Package_TO_SOT_SMD:SOT-23-5, symbol 74xGxx:74AUC1G79
- added U6, U7: 74LVC1G08, Package_TO_SOT_SMD:SOT-23-5, symbol 74xGxx:74LVC1G08
- added U9: 74LVC1G86, Package_TO_SOT_SMD:SOT-23-5, symbol 74xGxx:74LVC1G86
- U1: symbol 2021-07-26_01-49-48:MSP430F5171IDA -> gpsdo-rescue:MSP430F5171IDA-2021-07-26_01-49-48
Connections:
- net +3V3: now also J2.4 (Pin_4), C12.1, C13.1, C14.1, C15.1, J6.1 (Pin_1), U10.5 (VCC), U6.5 (VCC), U7.5 (VCC), U8.5 (VCC), U9.5 (VCC)
- net CLK_25M: now also U7.2, U8.2 (C)
- net GND: now also C12.2, C13.2, C14.2, C15.2, J6.4 (Pin_4), R8.1, R9.1, U10.3 (GND), U6.3 (GND), U7.3 (GND), U8.3 (GND), U9.3 (GND); no longer J3.3 (Pin_3), J3.4 (Pin_4)
- net gPPS: now also U1.16 (P1-7/PM_TD0-1), U1.27 (P3-0/PM_TEC1FLT2/PM_TD1-1), U10.1 (D); no longer U1.15 (P1-6/PM_TD0-0)
- net oPPS: now also U1.15 (P1-6/PM_TD0-0), U10.2 (C), U6.2, U8.4 (Q); no longer U1.16 (P1-7/PM_TD0-1)
- net SDA1: now reaches R7.1, U3.7 (SDA), U4.1 (SDA), U5.13 (SDAOUT1)
- net SCL1: now reaches R6.2, U3.8 (SCL), U4.6 (SCL), U5.14 (SCLOUT1)
- net SDA2: now reaches R5.1, U2.16 (SDA), U5.11 (SDAOUT2)
- net SCL2: now reaches R4.2, U2.17 (SCL), U5.16 (SCLOUT2)
- net gTXD: now reaches J5.1 (Pin_1), U2.2 (TXD)
- net gRXD: now reaches J5.2 (Pin_2), U2.3 (RXD)
- net SDA: now reaches R3.1, U1.9 (P1-4/PM_UCB0SIMO/PM_UCB0SDA/A4*/CB4), U5.12 (SDAIN)
- net SCL: now reaches R2.2, U1.10 (P1-5/PM_UCB0SOMI/PM_UCB0SCL/A5*/CB5), U5.15 (SCLIN)
- net EN1: now reaches U5.2 (ENABLE2)
- net EN1: now also U1.24 (P2-5/PM_TEC0FLT0/PM_TD0-1); no longer U1.23 (P2-4/PM_TEC0CLR/PM_TEC0FLT2_/PM_TD0-0)
- net EN2: now reaches U5.8 (ENABLE1)
- net EN2: now also U1.23 (P2-4/PM_TEC0CLR/PM_TEC0FLT2_/PM_TD0-0); no longer U1.24 (P2-5/PM_TEC0FLT0/PM_TD0-1)
- net uTXD: now reaches J4.1 (Pin_1), U1.6 (P1-1/PM_UCA0TXD/PM_UCA0SIMO/A1*/CB1)
- net uRXD: now reaches J4.2 (Pin_2), U1.7 (P1-2/PM_UCA0RXD/PM_UCA0SOMI/A2*/CB2)
- net dPPS: now reaches U1.18 (P2-1/PM___TD1-0)
- net dPPS: now also U10.4 (Q)
- net iPPS: now reaches U1.25 (P2-6/PM_TEC0FLT1/PM_TD0-2)
- net iPPS: now also U9.1
- net mPPS: now reaches U1.26 (P2-7/PM_TEC1CLR/PM_TEC1FLT1/PM_TD1-0)
- net mPPS: now also U9.2
- net SBWTCK: now reaches U1.35 (TEST/SBWTCK)
- net SBWTCK: now also J6.2 (Pin_2)
- net SBWTDIO: now reaches U1.36 (*RST/NMI/SBWTDIO)
- net SBWTDIO: now also J6.3 (Pin_3)
- net EN_CLK: now reaches U1.5 (P1-0/PM_UCA0CLK/PM_UCB0STE/A0*/CB0)
- net EN_CLK: now also R8.2, U7.1
- net EN_PPS: now reaches U1.8 (P1-3/PM_UCB0CLK/PM_UCA0STE/A3*/CB3)
- net EN_PPS: now also R9.2, U6.1
- net ePPS: no longer names the net of U1.17 (P2-0/PM_TD0-2)
- net ePPS: no longer J2.4 (Pin_4)
- new net: U8.1 (D), U9.4
- new net CLK: J3.3 (Pin_3), U7.4
- new net PPS: J3.4 (Pin_4), U6.4
