File: kicad/gpsdo.kicad_pcb (KiCad board)
At the start: 2 copper layers, 76.2 x 30.5 mm, 52 parts, among them J1 Conn_Coaxial, J2 Conn_01x04_Male, J3 Conn_01x04_Male, J4 Conn_01x04_Male, J5 Conn_01x04_Male, J6 Conn_01x04_Male, U1 MSP430F5171IDA, U10 74AUC1G79, U11 47L64, U12 47L64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

Commit message: fix SBW connection
Parts:
- added C23: 1n, Resistor_SMD:R_0603_1608Metric, F.Cu at (61.7, 31.0)
- added R11: 15k, Resistor_SMD:R_0603_1608Metric, F.Cu at (68.7, 27.8)
Routing:
- net GND: track 67.9 -> 70.1 mm, vias 51 -> 52
- net /SBWTCK: track 19.2 -> 19.7 mm
Changed lines of the file:
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@@
     (thickness 1.6)
     (drawings 4)
-    (tracks 521)
+    (tracks 530)
     (zones 0)
-    (modules 52)
+    (modules 54)
     (nets 57)
   )
@@
     (add_net mPPS)
     (add_net oPPS)
+  )
+  (module Resistor_SMD:R_0603_1608Metric (layer F.Cu)
+    (at 61.66 30.988 180)
+    (descr "Resistor SMD 0603 (1608 Metric), square (rectangular) end terminal, IPC_7351 nominal, (Body size source: http://www.tortai-tech.com/upload/download/2011102023233369053.pdf), generated with kicad-footprint-generator")
+    (tags resistor)
+    (attr smd)
+    (fp_text reference C23 (at 0 -1.43) (layer F.SilkS) hide
+      (effects (font (size 1 1) (thickness 0.15)))
+    )
+    (fp_text value 1n (at 0 1.43) (layer F.Fab) hide
+      (effects (font (size 1 1) (thickness 0.15)))
+    )
+    (fp_text user %R (at 0 0) (layer F.Fab)
+      (effects (font (size 0.4 0.4) (thickness 0.06)))
+    )
+    (fp_line (start 1.48 0.73) (end -1.48 0.73) (layer F.CrtYd) (width 0.05))
+    (fp_line (start 1.48 -0.73) (end 1.48 0.73) (layer F.CrtYd) (width 0.05))
+    (fp_line (start -1.48 -0.73) (end 1.48 -0.73) (layer F.CrtYd) (width 0.05))
+    (fp_line (start -1.48 0.73) (end -1.48 -0.73) (layer F.CrtYd) (width 0.05))
+    (fp_line (start -0.162779 0.51) (end 0.162779 0.51) (layer F.SilkS) (width 0.12))
+    (fp_line (start -0.162779 -0.51) (end 0.162779 -0.51) (layer F.SilkS) (width 0.12))
+    (fp_line (start 0.8 0.4) (end -0.8 0.4) (layer F.Fab) (width 0.1))
+    (fp_line (start 0.8 -0.4) (end 0.8 0.4) (layer F.Fab) (width 0.1))
+    (fp_line (start -0.8 -0.4) (end 0.8 -0.4) (layer F.Fab) (width 0.1))
+    (fp_line (start -0.8 0.4) (end -0.8 -0.4) (layer F.Fab) (width 0.1))
+    (pad 2 smd roundrect (at 0.7875 0 180) (size 0.875 0.95) (layers F.Cu F.Paste F.Mask) (roundrect_rratio 0.25)
+      (net 1 GND))
+    (pad 1 smd roundrect (at -0.7875 0 180) (size 0.875 0.95) (layers F.Cu F.Paste F.Mask) (roundrect_rratio 0.25)
+      (net 39 /SBWTDIO))
+    (model ${KISYS3DMOD}/Resistor_SMD.3dshapes/R_0603_1608Metric.wrl
+      (at (xyz 0 0 0))
+      (scale (xyz 1 1 1))
+      (rotate (xyz 0 0 0))
+    )
+  )
+  (module Resistor_SMD:R_0603_1608Metric (layer F.Cu)
+    (at 68.726463 27.823659 270)
+    (descr "Resistor SMD 0603 (1608 Metric), square (rectangular) end terminal, IPC_7351 nominal, (Body size source: http://www.tortai-tech.com/upload/download/2011102023233369053.pdf), generated with kicad-footprint-generator")
+    (tags resistor)
+    (attr smd)
+    (fp_text reference R11 (at 0 -1.43 90) (layer F.SilkS) hide
+      (effects (font (size 1 1) (thickness 0.15)))
+    )
+    (fp_text value 15k (at 0 1.43 90) (layer F.Fab) hide
+      (effects (font (size 1 1) (thickness 0.15)))
+    )
+    (fp_text user %R (at 0 0 90) (layer F.Fab)
+      (effects (font (size 0.4 0.4) (thickness 0.06)))
+    )
+    (fp_line (start 1.48 0.73) (end -1.48 0.73) (layer F.CrtYd) (width 0.05))
+    (fp_line (start 1.48 -0.73) (end 1.48 0.73) (layer F.CrtYd) (width 0.05))
+    (fp_line (start -1.48 -0.73) (end 1.48 -0.73) (layer F.CrtYd) (width 0.05))
+    (fp_line (start -1.48 0.73) (end -1.48 -0.73) (layer F.CrtYd) (width 0.05))
+    (fp_line (start -0.162779 0.51) (end 0.162779 0.51) (layer F.SilkS) (width 0.12))
+    (fp_line (start -0.162779 -0.51) (end 0.162779 -0.51) (layer F.SilkS) (width 0.12))
+    (fp_line (start 0.8 0.4) (end -0.8 0.4) (layer F.Fab) (width 0.1))
+    (fp_line (start 0.8 -0.4) (end 0.8 0.4) (layer F.Fab) (width 0.1))
+    (fp_line (start -0.8 -0.4) (end 0.8 -0.4) (layer F.Fab) (width 0.1))
+    (fp_line (start -0.8 0.4) (end -0.8 -0.4) (layer F.Fab) (width 0.1))
+    (pad 2 smd roundrect (at 0.7875 0 270) (size 0.875 0.95) (layers F.Cu F.Paste F.Mask) (roundrect_rratio 0.25)
+      (net 1 GND))
+    (pad 1 smd roundrect (at -0.7875 0 270) (size 0.875 0.95) (layers F.Cu F.Paste F.Mask) (roundrect_rratio 0.25)
+      (net 40 /SBWTCK))
+    (model ${KISYS3DMOD}/Resistor_SMD.3dshapes/R_0603_1608Metric.wrl
+      (at (xyz 0 0 0))
+      (scale (xyz 1 1 1))
+      (rotate (xyz 0 0 0))
+    )
   )
   (module RF_Shielding:Laird_Technologies_BMI-S-102_16.50x16.50mm (layer F.Cu)
@@
   (segment (start 84.263 52.259) (end 84.836 52.832) (width 0.762) (layer F.Cu) (net 1))
   (segment (start 84.201 52.259) (end 84.263 52.259) (width 0.762) (layer F.Cu) (net 1))
-  (segment (start 65.294 31.402302) (end 65.022853 31.131155) (width 0.254) (layer F.Cu) (net 2))
-  (segment (start 65.294 33.345) (end 65.294 31.402302) (width 0.254) (layer F.Cu) (net 2))
-  (segment (start 70.294 31.136583) (end 70.299428 31.131155) (width 0.254) (layer F.Cu) (net 2))
-  (segment (start 70.294 33.345) (end 70.294 31.136583) (width 0.254) (layer F.Cu) (net 2))
-  (segment (start 54.915 28.397) (end 55.372 27.94) (width 1.016) (layer F.Cu) (net 2))
-  (segment (start 54.915 30.48) (end 54.915 28.397) (width 1.016) (layer F.Cu) (net 2))
-  (via (at 67.056 52.832) (size 0.8) (drill 0.4) (layers F.Cu B.Cu) (net 2))
-  (via (at 68.58 51.308) (size 0.8) (drill 0.4) (layers F.Cu B.Cu) (net 2))
-  (segment (start 67.056 52.832) (end 68.58 51.308) (width 1.016) (layer B.Cu) (net 2))
-  (segment (start 73.406 26.924) (end 74.422 27.94) (width 1.016) (layer B.Cu) (net 2))
-  (segment (start 72.644 26.162) (end 73.406 26.924) (width 1.016) (layer B.Cu) (net 2))
-  (segment (start 59.69 26.162) (end 72.644 26.162) (width 1.016) (layer B.Cu) (net 2))
-  (segment (start 57.912 27.94) (end 59.69 26.162) (width 1.016) (layer B.Cu) (net 2))
   (via (at 89.408 43.18) (size 0.8) (drill 0.4) (layers F.Cu B.Cu) (net 1))
   (via (at 81.788 45.72) (size 0.8) (drill 0.4) (layers F.Cu B.Cu) (net 1))
@@
   (segment (start 85.344 52.324) (end 84.836 52.832) (width 1.016) (layer F.Cu) (net 1))
   (segment (start 86.009 52.324) (end 85.344 52.324) (width 1.016) (layer F.Cu) (net 1))
+  (segment (start 67.727159 28.611159) (end 67.564 28.448) (width 1.016) (layer F.Cu) (net 1))
+  (segment (start 68.726463 28.611159) (end 67.727159 28.611159) (width 1.016) (layer F.Cu) (net 1))
+  (segment (start 65.294 31.402302) (end 65.022853 31.131155) (width 0.254) (layer F.Cu) (net 2))
+  (segment (start 65.294 33.345) (end 65.294 31.402302) (width 0.254) (layer F.Cu) (net 2))
+  (segment (start 70.294 31.136583) (end 70.299428 31.131155) (width 0.254) (layer F.Cu) (net 2))
+  (segment (start 70.294 33.345) (end 70.294 31.136583) (width 0.254) (layer F.Cu) (net 2))
+  (segment (start 54.915 28.397) (end 55.372 27.94) (width 1.016) (layer F.Cu) (net 2))
+  (segment (start 54.915 30.48) (end 54.915 28.397) (width 1.016) (layer F.Cu) (net 2))
+  (via (at 67.056 52.832) (size 0.8) (drill 0.4) (layers F.Cu B.Cu) (net 2))
+  (via (at 68.58 51.308) (size 0.8) (drill 0.4) (layers F.Cu B.Cu) (net 2))
+  (segment (start 67.056 52.832) (end 68.58 51.308) (width 1.016) (layer B.Cu) (net 2))
+  (segment (start 73.406 26.924) (end 74.422 27.94) (width 1.016) (layer B.Cu) (net 2))
+  (segment (start 72.644 26.162) (end 73.406 26.924) (width 1.016) (layer B.Cu) (net 2))
+  (segment (start 59.69 26.162) (end 72.644 26.162) (width 1.016) (layer B.Cu) (net 2))
+  (segment (start 57.912 27.94) (end 59.69 26.162) (width 1.016) (layer B.Cu) (net 2))
+  (via (at 59.944 30.988) (size 0.8) (drill 0.4) (layers F.Cu B.Cu) (net 1))
+  (segment (start 60.8725 30.988) (end 59.944 30.988) (width 1.016) (layer F.Cu) (net 1))
   (segment (start 88.829938 36.646062) (end 89.408 36.068) (width 0.508) (layer F.Cu) (net 4))
   (segment (start 86.183678 36.646062) (end 88.829938 36.646062) (width 0.508) (layer F.Cu) (net 4))
@@
   (segment (start 62.794 29.363052) (end 65.941061 26.21599) (width 0.254) (layer F.Cu) (net 39))
   (segment (start 65.941061 26.21599) (end 77.77799 26.21599) (width 0.254) (layer F.Cu) (net 39))
-  (segment (start 62.794 33.345) (end 62.794 29.363052) (width 0.254) (layer F.Cu) (net 39))
   (segment (start 65.487052 26.67) (end 65.509526 26.647526) (width 0.254) (layer F.Cu) (net 39))
   (segment (start 64.7955 26.67) (end 65.487052 26.67) (width 0.254) (layer F.Cu) (net 39))
+  (segment (start 62.596 30.988) (end 62.794 30.79) (width 0.254) (layer F.Cu) (net 39))
+  (segment (start 62.4475 30.988) (end 62.596 30.988) (width 0.254) (layer F.Cu) (net 39))
+  (segment (start 62.794 30.79) (end 62.794 29.363052) (width 0.254) (layer F.Cu) (net 39))
+  (segment (start 62.794 33.345) (end 62.794 30.79) (width 0.254) (layer F.Cu) (net 39))
   (segment (start 63.294 29.505118) (end 66.129118 26.67) (width 0.254) (layer F.Cu) (net 40))
   (segment (start 63.294 33.345) (end 63.294 29.505118) (width 0.254) (layer F.Cu) (net 40))
   (segment (start 75.692 26.67) (end 76.962 27.94) (width 0.254) (layer F.Cu) (net 40))
   (segment (start 66.129118 26.67) (end 75.692 26.67) (width 0.254) (layer F.Cu) (net 40))
+  (segment (start 68.726463 26.67) (end 68.58 26.67) (width 0.254) (layer F.Cu) (net 40))
+  (segment (start 68.726463 27.036159) (end 68.726463 26.67) (width 0.254) (layer F.Cu) (net 40))
   (segment (start 72.41 46.756) (end 72.41 48.867) (width 0.254) (layer F.Cu) (net 41))
   (segment (start 72.062999 46.408999) (end 72.41 46.756) (width 0.254) (layer F.Cu) (net 41))
