File: kicad/ethernet.kicad_pcb (KiCad board)
At the start: 2 copper layers, 120 x 90 mm, 82 parts, among them J1 RJ45_Abracon_ARJP11A-MASA-B-A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, J2 Conn_Coaxial, J3 JTAG, J4 USB_C_Receptacle_USB2.0, J5 Conn_Coaxial, J6 Conn_Coaxial, Q1 BSO220N03MD, SW1 KSC701, SW2 KSC701, U1 MSP432E401Y, U2 MAX-8Q, U3 TPD4S014, U4 74AUC2G34, U5 74AUC2G34, U6 MAX40200AUK, Y1 NX3225GA-25.000M-STD-CRG-2

Commit message: board layout progress
Parts:
- removed D8: MBR0520L, Diode_SMD:D_SOD-123
- removed J4: USB_C_Receptacle_USB2.0, Connector_USB:USB_C_Receptacle_XKB_U262-16XN-4BVC11
- removed R18: 110k, Resistor_SMD:R_0805_2012Metric
- removed R21, R22: 220k, Resistor_SMD:R_0805_2012Metric
- removed R28, R29: 10k, Resistor_SMD:R_0805_2012Metric
- removed SW2: KSC701, Button_Switch_SMD:SW_Push_1P1T_NO_CK_KSC7xxJ
- added BT4: NiMH, Battery:BatteryHolder_Keystone_2466_1xAAA, F.Cu at (100.0, 62.0)
- added C25: 100n, Capacitor_SMD:C_0805_2012Metric, F.Cu at (110.0, 108.5)
- added D9: RB168L100DDTE25, Diode_SMD:D_SMA, F.Cu at (111.5, 53.0)
- added Q2: 3904, Package_TO_SOT_SMD:SOT-23, F.Cu at (122.8, 68.5)
- added U7: 4N25, Package_DIP:SMDIP-6_W9.53mm, F.Cu at (134.8, 68.5)
- C19: value 10n -> 100n
- C20: value 10n -> 10u
- C3: value 100n -> 10u
- D7: value MBR0520L -> HSMW-C170; footprint Diode_SMD:D_SOD-123 -> LED_SMD:LED_0805_2012Metric
- Q1: value BSO220N03MD -> 3904; footprint Package_SO:SOIC-8_3.9x4.9mm_P1.27mm -> Package_TO_SOT_SMD:SOT-23
- R12: value 10k -> 3k
- R15: value 5.1k -> 1k
- R17: value 110k -> 2.5k
- R6: value 49.9 -> 1k
- R7: value 5.1k -> 2.5k
- U3: value TPD4S014 -> TLV75733PDRV; footprint Package_SON:Texas_S-PWSON-N10 -> Package_SON:WSON-6-1EP_2x2mm_P0.65mm_EP1x1.6mm
- U6: value MAX40200AUK -> LT1634BCMS8-2.5; footprint Package_TO_SOT_SMD:SOT-23-5 -> Package_SO:MSOP-8_3x3mm_P0.65mm
- moved R6 80.6 mm to (110.2, 71.2), turned to 0 degrees
- moved R15 78.6 mm to (126.0, 71.8), turned to 90 degrees
- moved R7 72.5 mm to (114.2, 73.7)
- moved C3 72.2 mm to (106.2, 74.8), turned to -90 degrees
- moved C24 70.8 mm to (150.0, 118.2), turned to 180 degrees
- moved U3 59.9 mm to (103.5, 74.2), turned to 90 degrees
- moved U6 59.0 mm to (122.5, 75.0), turned to 90 degrees
- moved BT3 54.2 mm to (59.5, 74.0), turned to -90 degrees
- moved R12 52.4 mm to (114.8, 65.8)
- moved D7 37.3 mm to (114.2, 71.2)
- moved C23 36.9 mm to (110.0, 64.8), turned to 90 degrees
- moved R17 34.7 mm to (119.0, 64.9), turned to -90 degrees
- moved C22 34.3 mm to (106.5, 64.8), turned to 90 degrees
- moved TR1 33.8 mm to (122.5, 56.0), turned to 0 degrees
- moved BT2 30.4 mm to (74.5, 118.8), turned to 90 degrees
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Connections:
- BT3 pad 1: +BATT -> Net-(BT3-Pad1)
- C18 pad 2: Net-(C18-Pad2) -> Net-(U1-Pad1)
- C19 pad 2: Net-(C19-Pad2) -> +3V3
- C20 pad 2: Net-(C20-Pad2) -> +BATT
- C21 pad 1: Net-(C21-Pad1) -> unconnected-(C21-Pad1)
- C21 pad 2: Net-(C21-Pad2) -> unconnected-(C21-Pad2)
- C22 pad 2: +5VP -> +BATT
- C23 pad 2: +5VP -> +BATT
- C24 pad 1: Net-(C21-Pad1) -> -POE
- C24 pad 2: Net-(C21-Pad2) -> +POE
- C3 pad 1: Net-(C3-Pad1) -> GND
- C3 pad 2: GND -> +3V3
- D7 pad 1: +5VP -> Net-(U3-Pad4)
- D7 pad 2: Net-(D7-Pad2) -> +BATT
- J1 pad 10: unconnected-(J1-Pad10) -> -POE
- J1 pad 9: unconnected-(J1-Pad9) -> +POE
- Q1 pad 1: Net-(L2-Pad2) -> Net-(Q1-Pad1)
- Q1 pad 3: Net-(L2-Pad2) -> +BATT
- R12 pad 1: ~{WAKE} -> Net-(Q2-Pad1)
- R12 pad 2: +3V3 -> +BATT
- R15 pad 1: Net-(J4-PadB5) -> GND
- R15 pad 2: GND -> Net-(Q1-Pad2)
- R16 pad 1: Net-(C18-Pad2) -> Net-(U1-Pad1)
- R17 pad 1: Net-(C19-Pad2) -> GND
- R17 pad 2: GND -> Net-(Q2-Pad1)
- R19 pad 2: unconnected-(R19-Pad2) -> GPS_LED
- R20 pad 2: Net-(C18-Pad2) -> Net-(U1-Pad1)
- R24 pad 2: unconnected-(R24-Pad2) -> PLL_LED
- R26 pad 2: unconnected-(R26-Pad2) -> Net-(U1-Pad14)
- R27 pad 2: unconnected-(R27-Pad2) -> Net-(R27-Pad2)
- R6 pad 1: Net-(C3-Pad1) -> GND
- R6 pad 2: Net-(J4-PadS1) -> Net-(U3-Pad4)
- R7 pad 1: Net-(J4-PadA5) -> Net-(Q1-Pad1)
- R7 pad 2: GND -> +BATT
- TR1 pad 1: Net-(Q1-Pad4) -> Net-(D9-Pad2)
- TR1 pad 2: Net-(C21-Pad1) -> GND
- TR1 pad 3: Net-(Q1-Pad2) -> unconnected-(TR1-Pad3)
- TR1 pad 4: Net-(D8-Pad2) -> unconnected-(TR1-Pad4)
- TR1 pad 5: GND -> unconnected-(TR1-Pad5)
- TR1 pad 6: Net-(D7-Pad2) -> unconnected-(TR1-Pad6)
- U1 pad 1: unconnected-(U1-Pad1) -> Net-(U1-Pad1)
- U1 pad 11: unconnected-(U1-Pad11) -> +3V3
- U1 pad 116: unconnected-(U1-Pad116) -> +3V3
- U1 pad 117: unconnected-(U1-Pad117) -> +3V3
- U1 pad 118: unconnected-(U1-Pad118) -> +3V3
- U1 pad 119: unconnected-(U1-Pad119) -> +3V3
- U1 pad 12: Net-(C20-Pad2) -> +3V3
- U1 pad 120: unconnected-(U1-Pad120) -> +3V3
- U1 pad 121: unconnected-(U1-Pad121) -> +3V3
- U1 pad 123: unconnected-(U1-Pad123) -> +3V3
- U1 pad 124: unconnected-(U1-Pad124) -> +3V3
- U1 pad 125: unconnected-(U1-Pad125) -> +3V3
- U1 pad 126: unconnected-(U1-Pad126) -> +3V3
- U1 pad 128: unconnected-(U1-Pad128) -> +3V3
- U1 pad 13: Net-(C19-Pad2) -> +3V3
- U1 pad 14: Net-(C18-Pad2) -> Net-(U1-Pad14)
- U1 pad 15: unconnected-(U1-Pad15) -> Net-(R27-Pad2)
- U1 pad 18: unconnected-(U1-Pad18) -> +3V3
- U1 pad 19: unconnected-(U1-Pad19) -> +3V3
- U1 pad 2: unconnected-(U1-Pad2) -> +3V3
- U1 pad 20: unconnected-(U1-Pad20) -> +3V3
- U1 pad 21: unconnected-(U1-Pad21) -> +3V3
- U1 pad 22: unconnected-(U1-Pad22) -> +3V3
- U1 pad 23: unconnected-(U1-Pad23) -> +3V3
- U1 pad 24: unconnected-(U1-Pad24) -> +3V3
- U1 pad 25: unconnected-(U1-Pad25) -> +3V3
- U1 pad 27: unconnected-(U1-Pad27) -> +3V3
- U1 pad 29: unconnected-(U1-Pad29) -> PLL_LED
- U1 pad 3: unconnected-(U1-Pad3) -> +3V3
- U1 pad 30: unconnected-(U1-Pad30) -> GPS_LED
- U1 pad 4: unconnected-(U1-Pad4) -> +3V3
- U1 pad 5: unconnected-(U1-Pad5) -> +3V3
- U1 pad 6: unconnected-(U1-Pad6) -> +3V3
- U1 pad 64: ~{WAKE} -> GND
- U1 pad 66: unconnected-(U1-Pad66) -> GND
- U1 pad 71: unconnected-(U1-Pad71) -> +3V3
- U1 pad 72: unconnected-(U1-Pad72) -> +3V3
- U1 pad 73: unconnected-(U1-Pad73) -> +3V3
- U1 pad 74: unconnected-(U1-Pad74) -> +3V3
- U1 pad 93: D- -> unconnected-(U1-Pad93)
- U1 pad 94: D+ -> unconnected-(U1-Pad94)
- U1 pad 95: unconnected-(U1-Pad95) -> +3V3
- U1 pad 96: unconnected-(U1-Pad96) -> +3V3
- U3 pad 1: +5V -> +3V3
- U3 pad 2: +5V -> unconnected-(U3-Pad2)
- U3 pad 3: Net-(R29-Pad1) -> GND
- U3 pad 4: VUSB -> Net-(U3-Pad4)
- U3 pad 5: GND -> unconnected-(U3-Pad5)
- U3 pad 6: D- -> +BATT
- U3 pad 7: D+ -> GND
- U6 pad 1: +5VP -> (no net)
- U6 pad 2: GND -> (no net)
- U6 pad 3: +5VP -> (no net)
- U6 pad 4: unconnected-(U6-Pad4) -> GND
- U6 pad 5: +5V -> unconnected-(U6-Pad5)
Routing:
- net +BATT: track 10.1 -> 80.0 mm, vias 0 -> 2
- net D-: track 56.4 -> 0.00 mm, vias 2 -> 0
- net D+: track 55.8 -> 0.00 mm, vias 2 -> 0
- net Net-(U1-Pad14): track 0.00 -> 54.7 mm
- net Net-(R27-Pad2): track 0.00 -> 51.5 mm
- net Net-(BT2-Pad1): track 64.8 -> 15.0 mm
- net PLL_LED: track 0.00 -> 37.6 mm
- net Net-(C20-Pad2): track 31.9 -> 0.00 mm
- net ~{WAKE}: track 31.7 -> 0.00 mm
- net Net-(C19-Pad2): track 30.6 -> 0.00 mm
- net GPS_LED: track 0.00 -> 29.6 mm, vias 0 -> 2
- net Net-(C18-Pad2): track 29.6 -> 0.00 mm
- net +3V3: track 1.77 -> 26.9 mm, vias 2 -> 9
- net Net-(U1-Pad1): track 0.00 -> 23.0 mm
- net Net-(J4-PadS1): track 20.5 -> 0.00 mm
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- added copper zone on F.Cu, net +BATT
- removed copper zone on F.Cu, net +5VP
- removed copper zone on F.Cu, net /VBUS
Other:
- board size 120 x 90 mm -> 105 x 90 mm
- board text removed: "WAKE"

Commit message: board layout update
Parts:
- removed BT1, BT2, BT3, BT4: NiMH, Battery:BatteryHolder_Keystone_2466_1xAAA
- added C26: 10u, Capacitor_SMD:C_0805_2012Metric, F.Cu at (69.8, 83.8)
- added C27: 1n, Capacitor_SMD:C_0805_2012Metric, F.Cu at (65.8, 59.2)
- added J4: BATT, Connector_PinHeader_2.54mm:PinHeader_1x02_P2.54mm_Vertical, F.Cu at (74.5, 88.2)
- added J7: POE, Connector_PinHeader_2.54mm:PinHeader_1x02_P2.54mm_Vertical, F.Cu at (152.2, 92.0)
- added Q3: BSC340N08NS3G, Package_TO_SOT_SMD:TDSON-8-1, F.Cu at (72.5, 58.2)
- added Q4: MMBT5401L, Package_TO_SOT_SMD:SOT-23, F.Cu at (61.8, 54.8)
- added R18: 750m, Resistor_SMD:R_1206_3216Metric, F.Cu at (66.0, 57.0)
- added R21: 4.7k, Resistor_SMD:R_0805_2012Metric, F.Cu at (67.2, 53.8)
- moved C21 81.2 mm to (69.8, 87.2), turned to 180 degrees
- moved TR1 53.3 mm to (71.0, 69.8), turned to 90 degrees
- moved U7 52.4 mm to (83.5, 57.5), turned to 90 degrees
- moved D9 46.2 mm to (74.5, 80.8), turned to 90 degrees
- moved R17 40.0 mm to (79.9, 73.2), turned to 0 degrees
- moved R15 39.6 mm to (86.8, 66.2), turned to 180 degrees
- moved Q2 39.3 mm to (83.5, 69.5), turned to 90 degrees
- moved R12 36.0 mm to (80.8, 77.5), turned to -90 degrees
- moved C23 34.5 mm to (80.2, 82.2), turned to 180 degrees
- moved C22 33.6 mm to (80.2, 85.8), turned to 180 degrees
- moved U6 32.9 mm to (90.0, 69.8), turned to 180 degrees
- moved Q1 32.1 mm to (86.2, 74.0), turned to -90 degrees
- moved J3 29.7 mm to (110.9, 56.8), turned to 90 degrees
- moved D7 28.8 mm to (86.2, 78.1), turned to 90 degrees
- moved SW1 28.5 mm to (130.0, 55.5)
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Connections:
- net -POE renamed Net-(C24-Pad1)
- C21 pad 1: unconnected-(C21-Pad1) -> +BATT
- C21 pad 2: unconnected-(C21-Pad2) -> GND
- C24 pad 2: +POE -> Net-(C24-Pad2)
- D9 pad 2: Net-(D9-Pad2) -> Net-(TR1-Pad3)
- J1 pad 9: +POE -> Net-(C24-Pad2)
- TR1 pad 1: Net-(D9-Pad2) -> unconnected-(TR1-Pad1)
- TR1 pad 3: unconnected-(TR1-Pad3) -> Net-(TR1-Pad3)
- TR1 pad 4: unconnected-(TR1-Pad4) -> /PSW
- TR1 pad 6: unconnected-(TR1-Pad6) -> +POE
Routing:
- net +BATT: track 80.0 -> 30.9 mm, vias 2 -> 0
- net Net-(BT2-Pad1): track 15.0 -> 0.00 mm
- net Net-(BT1-Pad1): track 15.0 -> 0.00 mm
- net Net-(BT3-Pad1): track 13.7 -> 0.00 mm
- net Net-(C24-Pad2): track 0.00 -> 11.5 mm
- net Net-(J3-Pad2): track 8.79 -> 19.5 mm, vias 1 -> 0
- net Net-(J3-Pad6): track 7.99 -> 17.2 mm
- net +POE: track 8.66 -> 0.00 mm
- net ~{RST}: track 45.0 -> 36.6 mm
- net Net-(J3-Pad4): track 8.78 -> 16.1 mm, vias 1 -> 0
- net Net-(C18-Pad2): track 23.0 -> 17.5 mm
- net Net-(J3-Pad8): track 9.80 -> 13.7 mm
- net Net-(TR1-Pad3): track 0.00 -> 3.78 mm
- net Net-(D9-Pad2): track 2.82 -> 0.00 mm
- net Net-(C24-Pad1): track 11.9 -> 13.8 mm
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- added copper zone on F.Cu, net +POE
- added copper zone on B.Cu, net -POE
- added copper zone on F.Cu, net -POE
- added copper zone on F.Cu, net /ISENSE
- added copper zone on F.Cu, net /PSW
Other:
- board size 105 x 90 mm -> 105 x 62.5 mm
- board text added: "HEATSINK"

Commit message: finishing board layout
Parts:
- added C28: 100n, Capacitor_SMD:C_0805_2012Metric, F.Cu at (71.0, 91.8)
- added C29: 10u, Capacitor_SMD:C_0805_2012Metric, F.Cu at (61.5, 81.0)
- added C30: 10u, Capacitor_SMD:C_0805_2012Metric, F.Cu at (63.8, 81.0)
- added C31: 100n, Capacitor_SMD:C_0805_2012Metric, F.Cu at (57.8, 87.8)
- added D8: BZX84C12VLY, Diode_SMD:D_SOT-23_ANK, F.Cu at (62.0, 85.2)
- added J8: POE+, Connector_Pin:Pin_D0.9mm_L10.0mm_W2.4mm_FlatFork, F.Cu at (61.5, 77.5)
- added J9: POE-, Connector_Pin:Pin_D0.9mm_L10.0mm_W2.4mm_FlatFork, F.Cu at (67.8, 67.5)
- added Q10: 3904, Package_TO_SOT_SMD:SOT-23, F.Cu at (68.0, 91.8)
- added Q11: 3904, Package_TO_SOT_SMD:SOT-23, F.Cu at (62.0, 91.8)
- added Q12: 3906, Package_TO_SOT_SMD:SOT-23, F.Cu at (58.2, 91.8)
- added Q13: 3904, Package_TO_SOT_SMD:SOT-23, F.Cu at (52.8, 89.8)
- added Q5: 3904, Package_TO_SOT_SMD:SOT-23, F.Cu at (70.0, 81.0)
- added Q6: 3906, Package_TO_SOT_SMD:SOT-23, F.Cu at (66.5, 81.0)
- added Q7: 3904, Package_TO_SOT_SMD:SOT-23, F.Cu at (58.0, 84.0)
- added Q8: 3906, Package_TO_SOT_SMD:SOT-23, F.Cu at (70.0, 85.2)
- added Q9: 3904, Package_TO_SOT_SMD:SOT-23, F.Cu at (66.5, 85.2)
- added R22: 150k, Resistor_SMD:R_0805_2012Metric, F.Cu at (55.0, 85.2)
- added R28: 150k, Resistor_SMD:R_0805_2012Metric, F.Cu at (68.2, 88.5)
- added R29: 1k, Resistor_SMD:R_0805_2012Metric, F.Cu at (64.6, 88.5)
- added R30: 1k, Resistor_SMD:R_0805_2012Metric, F.Cu at (65.0, 91.8)
- added R31: 100, Resistor_SMD:R_0805_2012Metric, F.Cu at (52.0, 85.9)
- added R32: 10k, Resistor_SMD:R_0805_2012Metric, F.Cu at (54.5, 92.8)
- added R33: 10k, Resistor_SMD:R_0805_2012Metric, F.Cu at (55.5, 90.0)
- added R34: 10k, Resistor_SMD:R_0805_2012Metric, F.Cu at (61.0, 88.5)
- moved U3 33.3 mm to (88.8, 55.5), turned to -90 degrees
- moved C3 31.2 mm to (86.0, 55.0), turned to 90 degrees
- moved C19 29.2 mm to (83.5, 55.0), turned to 90 degrees
- moved C20 29.0 mm to (87.5, 58.5), turned to 0 degrees
- moved Q4 28.0 mm to (53.5, 81.5)
- moved R21 27.3 mm to (53.8, 77.5), turned to 90 degrees
- moved U7 26.3 mm to (57.5, 61.2), turned to 180 degrees
- moved U6 25.2 mm to (69.8, 54.8), turned to -90 degrees
- moved R7 24.4 mm to (78.0, 56.1), turned to 0 degrees
- moved J4 24.1 mm to (88.8, 68.8), turned to 90 degrees
- moved R6 23.9 mm to (82.0, 58.5), turned to 180 degrees
- moved R18 23.6 mm to (56.8, 78.8), turned to 90 degrees
- moved R15 22.1 mm to (66.2, 58.0), turned to -90 degrees
- moved C22 22.0 mm to (85.8, 64.5), turned to -90 degrees
- moved C21 21.4 mm to (87.2, 75.0), turned to -90 degrees
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Connections:
- Q3 pad 4: unconnected-(Q3-Pad4) -> Net-(Q3-Pad4)
- Q4 pad 3: unconnected-(Q4-Pad3) -> Net-(Q9-Pad1)
- U7 pad 4: unconnected-(U7-Pad4) -> -POE
- U7 pad 5: unconnected-(U7-Pad5) -> Net-(U7-Pad5)
Routing:
- net Net-(U7-Pad5): track 0.00 -> 41.2 mm
- net Net-(Q9-Pad1): track 0.00 -> 18.3 mm, vias 0 -> 2
- net +POE: track 0.00 -> 15.6 mm
- net Net-(Q3-Pad4): track 0.00 -> 14.8 mm
- net +BATT: track 30.9 -> 17.5 mm
- net /ISENSE: track 0.00 -> 12.1 mm
- net Net-(Q10-Pad1): track 0.00 -> 11.9 mm
- net Net-(Q5-Pad1): track 0.00 -> 11.0 mm
- net -POE: track 0.00 -> 10.2 mm, vias 4 -> 26
- net Net-(Q7-Pad1): track 0.00 -> 7.79 mm
- net /VDRV: track 0.00 -> 5.19 mm
- net Net-(Q13-Pad1): track 0.00 -> 3.95 mm
- net Net-(Q12-Pad3): track 0.00 -> 3.07 mm
- net Net-(Q13-Pad3): track 0.00 -> 2.86 mm
- net Net-(Q10-Pad3): track 0.00 -> 2.59 mm
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- added copper zone on F.Cu, net /VDRV
Other:
- board size 105 x 62.5 mm -> 92 x 62.5 mm
